Commit message: update robot model

File: robot_description/urdf/slam_robot.urdf (robot description, URDF)
Before this commit: robot slam_robot, 6 links, 5 joints
Links:
- added link base_footprint
- added link caster_link, mass 0.500; collision sphere radius=0.05; visual sphere radius=0.05
- link base_link: mass None -> 0.500
- link left_wheel_link: mass None -> 0.500; geometry collision cylinder length=0.05 radius=0.1; visual cylinder length=${WHEEL_LENGTH} radius=${WHEEL_RADIUS}
- link right_wheel_link: mass None -> 0.500; geometry collision cylinder length=0.05 radius=0.1; visual cylinder length=${WHEEL_LENGTH} radius=${WHEEL_RADIUS}
Joints:
- added joint base_link_joint: type fixed, parent base_footprint, child base_link, origin xyz=0 0 0.100
- added joint caster_joint: type fixed, parent base_link, child caster_link, origin xyz=0.150 0 -0.050

Commit message: add xtion_pro_live

File: robot_description/urdf/slam_robot.urdf (robot description, URDF)
Before this commit: robot slam_robot, 8 links, 7 joints
Links:
- removed link base_footprint
- removed link caster_link
- removed link left_wheel_link
- removed link pico_flexx_depth_frame
- removed link pico_flexx_link
- removed link pico_flexx_link_optical_frame
- removed link right_wheel_link
Joints:
- removed joint base_link_joint
- removed joint caster_joint
- removed joint left_wheel_joint
- removed joint pico_flexx_base_joint
- removed joint pico_flexx_depth_joint
- removed joint pico_flexx_joint
- removed joint right_wheel_joint
