Commit message: add body

File: robot_description/urdf/sensors/xtion_pro_live/xtion_pro_live.urdf.xacro (robot description, xacro)
@@ -4,5 +4,5 @@
   <xacro:include filename="$(find robot_description)/urdf/slambot_gazebo.urdf.xacro"/>
   -->
-  <xacro:include filename="$(find robot_description)/urdf/slambot_properties.urdf.xacro"/>
+  <xacro:include filename="$(find robot_description)/urdf/common_properties.urdf.xacro"/>
   <!-- Xacro properties -->
   <xacro:property name="M_SCALE" value="0.001"/>

File: robot_description/urdf/slam_robot.urdf (robot description, URDF)
Before this commit: robot slambot, 1 links, 0 joints
Links:
- removed link base_link
- added link base_footprint

File: robot_description/urdf/slambot_properties.urdf.xacro (robot description, xacro)
@@ -2,4 +2,7 @@
 <robot xmlns:xacro="http://ros.org/wiki/xacro">
   <xacro:include filename="$(find robot_description)/urdf/common_properties.urdf.xacro"/>
+  <xacro:include filename="$(find robot_description)/urdf/body/body.urdf.xacro"/>
+  <xacro:include filename="$(find robot_description)/urdf/sensors/xtion_pro_live/xtion_pro_live.urdf.xacro"/>
+  <xacro:include filename="$(find robot_description)/urdf/wheel/wheel.urdf.xacro"/>
   <xacro:property name="cam_px" value="-0.087" />
 <!--	<xacro:property name="cam_py" value="-0.0125" /> Y varies for different configurations. get sets in sensors_urdf -->
@@ -8,8 +11,3 @@
   <xacro:property name="cam_op" value="0" />
   <xacro:property name="cam_oy" value="0" />
-  <!-- Wheel property -->
-  <xacro:property name="wheel_radius" value="0.0249" />
-  <xacro:property name="wheel_length" value="0.008" />
-  <xacro:property name="tread_width" value="0.1500" />
-  <property name="wheel_mass" value="0.0113"/>
 </robot>

File: robot_description/urdf/wheel/wheel.urdf.xacro (robot description, xacro)
@@ -3,5 +3,8 @@
   <xacro:include filename="$(find robot_description)/urdf/wheel/wheel.transmission.xacro"/>
   <xacro:include filename="$(find robot_description)/urdf/wheel/wheel.gazebo.xacro"/>
-    <xacro:include filename="$(find robot_description)/urdf/slambot_properties.urdf.xacro"/>
+  <xacro:include filename="$(find robot_description)/urdf/common_properties.urdf.xacro"/>
+  <xacro:property name="wheel_radius" value="0.0249" />
+  <xacro:property name="wheel_length" value="0.008" />
+  <xacro:property name="wheel_mass" value="0.0113"/>
   <!-- <property name="wheel_radius" value="0.0239"/> -->
   <xacro:macro name="wheel" params="prefix parent *joint_origin *joint_axis">

Commit message: update

File: robot_description/urdf/sensors/xtion_pro_live/xtion_pro_live.urdf.xacro (robot description, xacro)
@@ -11,13 +11,13 @@
   <xacro:property name="xtion_pro_live_cam_rel_rgb_py"   value="-0.0220" />
   <!-- Parameterised in part by the values in slambot_properties.urdf.xacro -->
-  <xacro:macro name="sensor_xtion_pro_live" params="parent name">
-    <joint name="${name}_rgb_joint" type="fixed">
+  <xacro:macro name="sensor_xtion_pro_live" params="prefix parent">
+    <joint name="${prefix}_rgb_joint" type="fixed">
       <origin xyz="${cam_px} ${xtion_pro_live_cam_py} ${cam_pz}"
               rpy="${cam_or} ${cam_op} ${cam_oy}"/>
       <parent link="${parent}"/>
-      <child link="${name}_rgb_frame" />
+      <child link="${prefix}_rgb_frame" />
     </joint>
-    <link name="${name}_rgb_frame"/>
-    <link name="${name}_link">
+    <link name="${prefix}_rgb_frame"/>
+    <link name="${prefix}_link">
       <visual>
         <origin xyz="-0.015 0.0035 0.004"
@@ -43,34 +43,34 @@
     </link>
     <!-- Xtion RGB sensor physical attachment -->
-    <joint name="${name}_joint" type="fixed">
+    <joint name="${prefix}_joint" type="fixed">
       <origin xyz="0 ${xtion_pro_live_cam_rel_rgb_py} 0"
               rpy="0 0 0"/>
-      <parent link="${name}_rgb_frame"/>
-      <child link="${name}_link"/>
+      <parent link="${prefix}_rgb_frame"/>
+      <child link="${prefix}_link"/>
     </joint>
     <!-- Xtion RGB sensor frame -->
-    <joint name="${name}_rgb_optical_joint" type="fixed">
+    <joint name="${prefix}_rgb_optical_joint" type="fixed">
       <origin xyz="0 0 0"
               rpy="${-M_PI/2} 0 ${-M_PI/2}" />
-      <parent link="${name}_rgb_frame" />
-      <child link="${name}_rgb_optical_frame" />
+      <parent link="${prefix}_rgb_frame" />
+      <child link="${prefix}_rgb_optical_frame" />
     </joint>
-    <link name="${name}_rgb_optical_frame"/>
+    <link name="${prefix}_rgb_optical_frame"/>
     <!-- Xtion IR sensor physical attachment -->
-    <joint name="${name}_ir_joint" type="fixed">
+    <joint name="${prefix}_ir_joint" type="fixed">
       <origin xyz="0 ${xtion_pro_live_ir_rel_rgb_py} 0"
               rpy="0 0 0" />
-      <parent link="${name}_rgb_frame" />
-      <child link="${name}_ir_frame" />
+      <parent link="${prefix}_rgb_frame" />
+      <child link="${prefix}_ir_frame" />
     </joint>
-    <link name="${name}_ir_frame"/>
+    <link name="${prefix}_ir_frame"/>
     <!-- Xtion IR sensor frame -->
-    <joint name="${name}_ir_optical_joint" type="fixed">
+    <joint name="${prefix}_ir_optical_joint" type="fixed">
       <origin xyz="0 0 0"
               rpy="${-M_PI/2} 0 ${-M_PI/2}" />
-      <parent link="${name}_ir_frame" />
-      <child link="${name}_ir_optical_frame" />
+      <parent link="${prefix}_ir_frame" />
+      <child link="${prefix}_ir_optical_frame" />
     </joint>
-    <link name="${name}_ir_optical_frame"/>
+    <link name="${prefix}_ir_optical_frame"/>
     <!-- RGBD sensor for simulation, same as Kinect -->
     <slambot_sim_3dsensor/>

Commit message: update

File: robot_description/urdf/sensors/xtion_pro_live/xtion_pro_live.urdf.xacro (robot description, xacro)
@@ -7,12 +7,11 @@
   <!-- Xacro properties -->
   <xacro:property name="M_SCALE" value="0.001"/>
-  <xacro:property name="xtion_pro_live_cam_py" value="0.0205"/>
   <xacro:property name="xtion_pro_live_ir_rel_rgb_py" value="0.0270" />
   <xacro:property name="xtion_pro_live_cam_rel_rgb_py"   value="-0.0220" />
   <!-- Parameterised in part by the values in slambot_properties.urdf.xacro -->
-  <xacro:macro name="sensor_xtion_pro_live" params="prefix parent">
+  <xacro:macro name="sensor_xtion_pro_live" params="prefix parent *joint_origin *joint_axis">
     <joint name="${prefix}_rgb_joint" type="fixed">
-      <origin xyz="${cam_px} ${xtion_pro_live_cam_py} ${cam_pz}"
-              rpy="${cam_or} ${cam_op} ${cam_oy}"/>
+      <insert_block name="joint_origin"/>
+      <insert_block name="joint_axis"/>
       <parent link="${parent}"/>
       <child link="${prefix}_rgb_frame" />
@@ -21,5 +20,6 @@
     <link name="${prefix}_link">
       <visual>
-        <origin xyz="-0.015 0.0035 0.004"
+<!--         <origin xyz="-0.015 0.0035 0.004" -->
+        <origin xyz="0 0 0"
                 rpy="0 0 0"/>
         <geometry>

File: robot_description/urdf/slambot_properties.urdf.xacro (robot description, xacro)
@@ -5,9 +5,3 @@
   <xacro:include filename="$(find robot_description)/urdf/sensors/xtion_pro_live/xtion_pro_live.urdf.xacro"/>
   <xacro:include filename="$(find robot_description)/urdf/wheel/wheel.urdf.xacro"/>
-  <xacro:property name="cam_px" value="-0.087" />
-<!--	<xacro:property name="cam_py" value="-0.0125" /> Y varies for different configurations. get sets in sensors_urdf -->
-  <xacro:property name="cam_pz" value="0.2870" />
-  <xacro:property name="cam_or" value="0" />
-  <xacro:property name="cam_op" value="0" />
-  <xacro:property name="cam_oy" value="0" />
 </robot>
