Commit message: update

File: robot_description/urdf/body/body.urdf.xacro (robot description, xacro)
@@ -7,5 +7,5 @@
   <xacro:property name="body_z" value="0.046" />
   <xacro:property name="velocity_scale_factor" value="1.0"/>
-  <xacro:macro name="base" params="parent *joint_origin">
+  <xacro:macro name="body" params="parent *joint_origin">
   <joint name="base_joint" type="fixed">
     <insert_block name="joint_origin"/>

File: robot_description/urdf/sensors/xtion_pro_live/xtion_pro_live.urdf.xacro (robot description, xacro)
@@ -12,5 +12,4 @@
   <!-- Parameterised in part by the values in slambot_properties.urdf.xacro -->
   <xacro:macro name="sensor_xtion_pro_live" params="parent name">
-    <!-- base link -->
     <joint name="${name}_rgb_joint" type="fixed">
       <origin xyz="${cam_px} ${xtion_pro_live_cam_py} ${cam_pz}"

File: robot_description/urdf/slam_robot.urdf (robot description, URDF)
Before this commit: robot slambot, 1 links, 0 joints
Links:
- added link base_body
Joints:
- added joint base_footprint_joint: type fixed, parent base_footprint, child base_body, origin xyz=0 0 ${ofs_foot}

Commit message: update

File: robot_description/urdf/body/body.urdf.xacro (robot description, xacro)
@@ -2,8 +2,14 @@
 <robot xmlns:xacro="http://ros.org/wiki/xacro">
   <xacro:include filename="$(find robot_description)/urdf/common_properties.urdf.xacro"/>
+  <xacro:include filename="$(find robot_description)/urdf/body/caster_board.urdf.xacro" />
   <xacro:property name="tread_width" value="0.1500" />
+  <!-- Base Body -->
   <xacro:property name="body_x" value="0.210" />
   <xacro:property name="body_y" value="0.160" />
-  <xacro:property name="body_z" value="0.046" />
+  <xacro:property name="body_z" value="0.003" />
+  <xacro:property name="spacer_len27" value="0.027" />
+  <xacro:property name="spacer_rud27" value="0.003" />
+  <xacro:property name="spacer_len40" value="0.040" />
+  <xacro:property name="spacer_rud40" value="0.003" />
   <xacro:property name="velocity_scale_factor" value="1.0"/>
   <xacro:macro name="body" params="parent *joint_origin">
@@ -14,4 +20,5 @@
   </joint>
   <!-- Robot Body -->
+  <!-- Base Board -->
   <link name="base_link">
     <visual>
@@ -19,4 +26,7 @@
         <box size="${body_x} ${body_y} ${body_z}"/>
       </geometry>
+      <material name="white">
+        <color rgba="1 1 1 1"/>
+      </material>
     </visual>
     <collision>
@@ -31,4 +41,172 @@
     </inertial>
   </link>
+  <!-- Upper Board -->
+  <joint name="upper_board_joint" type="fixed">
+    <parent link="base_link"/>
+    <child link="upper_board"/>
+    <origin xyz="0 0 ${body_z/2 + spacer_len40 + body_z/2}"
+            rpy="0 0 0"/>
+    <axis xyz="0 0 0"/>
+  </joint>
+  <link name="upper_board">
+    <visual>
+      <geometry>
+        <box size="${body_x} ${body_y} ${body_z}"/>
+      </geometry>
+      <material name="white">
+        <color rgba="1 1 1 1"/>
+      </material>
+    </visual>
+    <collision>
+      <geometry>
+        <box size="${body_x} ${body_y} ${body_z}"/>
+      </geometry>
+    </collision>
+    <inertial>
+      <origin xyz="0 0 0"/>
+      <mass value="0.500"/>
+      <inertia ixx="0.0020833333" ixy="0" ixz="0" iyy="0.0070833333" iyz="0" izz="0.0083333333"/>
+    </inertial>
+  </link>
+  <!-- Front caster_board -->
+  <xacro:caster_board prefix="front" parent="base_link">
+    <origin xyz="${body_x/2 - caster_board_x/2} 0 -${body_z/2 + spacer_len27 + body_z/2 }"
+            rpy="0 0 0"/>
+    <axis xyz="0 0 0"/>
+  </xacro:caster_board>
+  <!-- Rear caster_board -->
+  <xacro:caster_board prefix="rear" parent="base_link">
+    <origin xyz="-${body_x/2 - caster_board_x/2} 0 -${body_z/2 + spacer_len27 + body_z/2 }"
+            rpy="0 0 0"/>
+    <axis xyz="0 0 0"/>
+  </xacro:caster_board>
+  <!-- Spacer_1 -->
+  <joint name="base_link_spacer_joint_1" type="fixed">
+    <parent link="base_link"/>
+    <child link="base_link_spacer_1"/>
+    <origin xyz="${body_x/2} ${body_y/2} 0"
+            rpy="0 0 0"/>
+    <axis xyz="0 0 0"/>
+  </joint>
+  <link name="base_link_spacer_1">
+    <visual>
+      <origin xyz="-${spacer_rud40} -${spacer_rud40} ${spacer_len40/2 + body_z/2}"
+              rpy="0 0 0"/>
+      <geometry>
+        <cylinder length="${spacer_len40}" radius="${spacer_rud40}"/>
+      </geometry>
+      <material name="white">
+        <color rgba="1 1 1 1"/>
+      </material>
+    </visual>
+    <collision>
+      <origin xyz="-${spacer_rud40} -${spacer_rud40} ${spacer_len40/2 + body_z/2}"
+              rpy="0 0 0"/>
+      <geometry>
+        <cylinder length="${spacer_len40}" radius="${spacer_rud40}"/>
+      </geometry>
+    </collision>
+    <inertial>
+      <origin rpy="0 0 0" xyz="0 0 0.5"/>
+      <mass value="0.1"/>
+      <inertia ixx="0.1" ixy="0" ixz="0" iyy="0.1" iyz="0" izz="0.1"/>
+    </inertial>
+  </link>
+  <!-- Spacer_2 -->
+  <joint name="base_link_spacer_joint_2" type="fixed">
+    <parent link="base_link"/>
+    <child link="base_link_spacer_2"/>
+    <origin xyz="${body_x/2} -${body_y/2} 0"
+            rpy="0 0 0"/>
+    <axis xyz="0 0 0"/>
+  </joint>
+  <link name="base_link_spacer_2">
+    <visual>
+      <origin xyz="-${spacer_rud40} ${spacer_rud40} ${spacer_len40/2 + body_z/2}"
+              rpy="0 0 0"/>
+      <geometry>
+        <cylinder length="${spacer_len40}" radius="${spacer_rud40}"/>
+      </geometry>
+      <material name="white">
+        <color rgba="1 1 1 1"/>
+      </material>
+    </visual>
+    <collision>
+      <origin xyz="-${spacer_rud40} ${spacer_rud40} ${spacer_len40/2 + body_z/2}"
+              rpy="0 0 0"/>
+      <geometry>
+        <cylinder length="${spacer_len40}" radius="${spacer_rud40}"/>
+      </geometry>
+    </collision>
+    <inertial>
+      <origin rpy="0 0 0" xyz="0 0 0.5"/>
+      <mass value="0.1"/>
+      <inertia ixx="0.1" ixy="0" ixz="0" iyy="0.1" iyz="0" izz="0.1"/>
+    </inertial>
+  </link>
+  <!-- Spacer_3 -->
+  <joint name="base_link_spacer_joint_3" type="fixed">
+    <parent link="base_link"/>
+    <child link="base_link_spacer_3"/>
+    <origin xyz="-${body_x/2} ${body_y/2} 0"
+            rpy="0 0 0"/>
+    <axis xyz="0 0 0"/>
+  </joint>
+  <link name="base_link_spacer_3">
+    <visual>
+      <origin xyz="${spacer_rud40} -${spacer_rud40} ${spacer_len40/2 + body_z/2}"
+              rpy="0 0 0"/>
+      <geometry>
+        <cylinder length="${spacer_len40}" radius="${spacer_rud40}"/>
+      </geometry>
+      <material name="white">
+        <color rgba="1 1 1 1"/>
+      </material>
+    </visual>
+    <collision>
+      <origin xyz="${spacer_rud40} -${spacer_rud40} ${spacer_len40/2 + body_z/2}"
+              rpy="0 0 0"/>
+      <geometry>
+        <cylinder length="${spacer_len40}" radius="${spacer_rud40}"/>
+      </geometry>
+    </collision>
+    <inertial>
+      <origin rpy="0 0 0" xyz="0 0 0.5"/>
+      <mass value="0.1"/>
+      <inertia ixx="0.1" ixy="0" ixz="0" iyy="0.1" iyz="0" izz="0.1"/>
+    </inertial>
+  </link>
+  <!-- Spacer_4 -->
+  <joint name="base_link_spacer_joint_4" type="fixed">
+    <parent link="base_link"/>
+    <child link="base_link_spacer_4"/>
+    <origin xyz="-${body_x/2} -${body_y/2} 0"
+            rpy="0 0 0"/>
+    <axis xyz="0 0 0"/>
+  </joint>
+  <link name="base_link_spacer_4">
+    <visual>
+      <origin xyz="${spacer_rud40} ${spacer_rud40} ${spacer_len40/2 + body_z/2}"
+              rpy="0 0 0"/>
+      <geometry>
+        <cylinder length="${spacer_len40}" radius="${spacer_rud40}"/>
+      </geometry>
+      <material name="white">
+        <color rgba="1 1 1 1"/>
+      </material>
+    </visual>
+    <collision>
+      <origin xyz="${spacer_rud40} ${spacer_rud40} ${spacer_len40/2 + body_z/2}"
+              rpy="0 0 0"/>
+      <geometry>
+        <cylinder length="${spacer_len40}" radius="${spacer_rud40}"/>
+      </geometry>
+    </collision>
+    <inertial>
+      <origin rpy="0 0 0" xyz="0 0 0.5"/>
+      <mass value="0.1"/>
+      <inertia ixx="0.1" ixy="0" ixz="0" iyy="0.1" iyz="0" izz="0.1"/>
+    </inertial>
+  </link>
   </xacro:macro>
 </robot>
