Commit message: chenge structure

File: slambot_sim/slambot_description/urdf/body/body.urdf.xacro (robot description, xacro)
@@ -1,6 +1,6 @@
 <?xml version="1.0"?>
 <robot xmlns:xacro="http://ros.org/wiki/xacro">
-  <xacro:include filename="$(find robot_description)/urdf/common_properties.urdf.xacro"/>
-  <xacro:include filename="$(find robot_description)/urdf/body/caster_board.urdf.xacro" />
+  <xacro:include filename="$(find slambot_description)/urdf/common_properties.urdf.xacro"/>
+  <xacro:include filename="$(find slambot_description)/urdf/body/caster_board.urdf.xacro" />
   <xacro:property name="tread_width" value="0.1500" />
   <!-- Base Body -->

File: slambot_sim/slambot_description/urdf/body/caster_board.urdf.xacro (robot description, xacro)
@@ -1,5 +1,5 @@
 <?xml version="1.0"?>
 <robot xmlns:xacro="http://ros.org/wiki/xacro">
-  <xacro:include filename="$(find robot_description)/urdf/common_properties.urdf.xacro"/>
+  <xacro:include filename="$(find slambot_description)/urdf/common_properties.urdf.xacro"/>
   <!-- Caster board -->
   <xacro:property name="caster_board_x" value="0.060" />

File: slambot_sim/slambot_description/urdf/sensors/xtion_pro_live/xtion_pro_live.urdf.xacro (robot description, xacro)
@@ -2,7 +2,7 @@
 <robot xmlns:xacro="http://ros.org/wiki/xacro">
   <!--
-  <xacro:include filename="$(find robot_description)/urdf/slambot_gazebo.urdf.xacro"/>
+  <xacro:include filename="$(find slabot_description)/urdf/slambot_gazebo.urdf.xacro"/>
   -->
-  <xacro:include filename="$(find robot_description)/urdf/common_properties.urdf.xacro"/>
+  <xacro:include filename="$(find slambot_description)/urdf/common_properties.urdf.xacro"/>
   <!-- Xacro properties -->
   <xacro:property name="M_SCALE" value="0.001"/>
@@ -24,5 +24,5 @@
                 rpy="0 0 0"/>
         <geometry>
-          <mesh filename="package://robot_description/urdf/sensors/xtion_pro_live/meshes/xtion_pro_camera.dae"/>
+          <mesh filename="package://slambot_description/urdf/sensors/xtion_pro_live/meshes/xtion_pro_camera.dae"/>
         </geometry>
       </visual>
@@ -86,5 +86,5 @@
         <origin xyz="0 0 0" rpy="${-M_PI/2} 0 0"/>
         <geometry>
-          <mesh filename="package://robot_description/meshes/sensors/xtion_pro_stack.dae"/>
+          <mesh filename="package://slabot_description/meshes/sensors/xtion_pro_stack.dae"/>
         </geometry>
       </visual>

File: slambot_sim/slambot_description/urdf/wheel/wheel.urdf.xacro (robot description, xacro)
@@ -1,7 +1,7 @@
 <?xml version="1.0"?>
 <robot xmlns:xacro="http://ros.org/wiki/xacro">
-  <xacro:include filename="$(find robot_description)/urdf/wheel/wheel.transmission.xacro"/>
-  <xacro:include filename="$(find robot_description)/urdf/wheel/wheel.gazebo.xacro"/>
-  <xacro:include filename="$(find robot_description)/urdf/common_properties.urdf.xacro"/>
+  <xacro:include filename="$(find slambot_description)/urdf/wheel/wheel.transmission.xacro"/>
+  <xacro:include filename="$(find slambot_description)/urdf/wheel/wheel.gazebo.xacro"/>
+  <xacro:include filename="$(find slambot_description)/urdf/common_properties.urdf.xacro"/>
   <xacro:property name="wheel_radius" value="0.0249" />
   <xacro:property name="wheel_length" value="0.008" />
@@ -21,5 +21,5 @@
     <visual>
       <geometry>
-        <mesh filename="package://robot_description/urdf/wheel/meshes/RasPiMouse_wheel.dae"/>
+        <mesh filename="package://slambot_description/urdf/wheel/meshes/RasPiMouse_wheel.dae"/>
       </geometry>
     </visual>
@@ -28,5 +28,5 @@
         <geometry>
           <!-- <cylinder radius="${wheel_radius}" length="${wheel_length}"/> -->
-          <mesh filename="package://robot_description/urdf/wheel/meshes/RasPiMouse_wheel.dae"/>
+          <mesh filename="package://slambot_description/urdf/wheel/meshes/RasPiMouse_wheel.dae"/>
         </geometry>
     </collision>

Commit message: update

File: slambot_sim/slambot_description/urdf/body/body.urdf.xacro (robot description, xacro)
@@ -17,9 +17,39 @@
     <insert_block name="joint_origin"/>
     <parent link="${parent}"/>
-    <child link="base_link"/>
+    <child link="base_body"/>
   </joint>
   <!-- Robot Body -->
   <!-- Base Board -->
-  <link name="base_link">
+  <link name="base_body">
+    <visual>
+      <origin xyz="0 0 ${body_z/2}"/>
+      <geometry>
+        <box size="${body_x} ${body_y} ${body_z}"/>
+      </geometry>
+      <material name="white">
+        <color rgba="1 1 1 1"/>
+      </material>
+    </visual>
+    <collision>
+      <origin xyz="0 0 ${body_z/2}"/>
+      <geometry>
+        <box size="${body_x} ${body_y} ${body_z}"/>
+      </geometry>
+    </collision>
+    <inertial>
+      <origin xyz="0 0 ${body_z/2}"/>
+      <mass value="0.500"/>
+      <inertia ixx="0.0020833333" ixy="0" ixz="0" iyy="0.0070833333" iyz="0" izz="0.0083333333"/>
+    </inertial>
+  </link>
+  <!-- Upper Board -->
+  <joint name="upper_board_joint" type="fixed">
+    <parent link="base_body"/>
+    <child link="upper_board"/>
+    <origin xyz="0 0 ${body_z + spacer_len40 + body_z/2}"
+            rpy="0 0 0"/>
+    <axis xyz="0 0 0"/>
+  </joint>
+  <link name="upper_board">
     <visual>
       <geometry>
@@ -41,72 +71,45 @@
     </inertial>
   </link>
-  <!-- Upper Board -->
-  <joint name="upper_board_joint" type="fixed">
-    <parent link="base_link"/>
-    <child link="upper_board"/>
-    <origin xyz="0 0 ${body_z/2 + spacer_len40 + body_z/2}"
-            rpy="0 0 0"/>
-    <axis xyz="0 0 0"/>
-  </joint>
-  <link name="upper_board">
-    <visual>
-      <geometry>
-        <box size="${body_x} ${body_y} ${body_z}"/>
-      </geometry>
-      <material name="white">
-        <color rgba="1 1 1 1"/>
-      </material>
-    </visual>
-    <collision>
-      <geometry>
-        <box size="${body_x} ${body_y} ${body_z}"/>
-      </geometry>
-    </collision>
-    <inertial>
-      <origin xyz="0 0 0"/>
-      <mass value="0.500"/>
-      <inertia ixx="0.0020833333" ixy="0" ixz="0" iyy="0.0070833333" iyz="0" izz="0.0083333333"/>
-    </inertial>
-  </link>
   <!-- Front caster_board -->
-  <xacro:caster_board prefix="front" parent="base_link">
-    <origin xyz="${body_x/2 - caster_board_x/2} 0 -${body_z/2 + spacer_len27 + body_z/2 }"
+  <xacro:caster_board prefix="front" parent="base_body">
+    <origin xyz="${body_x/2 - caster_board_x/2} 0 -${spacer_len27}"
             rpy="0 0 0"/>
     <axis xyz="0 0 0"/>
   </xacro:caster_board>
   <!-- Rear caster_board -->
-  <xacro:caster_board prefix="rear" parent="base_link">
-    <origin xyz="-${body_x/2 - caster_board_x/2} 0 -${body_z/2 + spacer_len27 + body_z/2 }"
+  <xacro:caster_board prefix="rear" parent="base_body">
+    <origin xyz="-${body_x/2 - caster_board_x/2} 0 -${spacer_len27}"
             rpy="0 0 0"/>
     <axis xyz="0 0 0"/>
   </xacro:caster_board>
   <!-- Spacer_1 -->
-  <joint name="base_link_spacer_joint_1" type="fixed">
-    <parent link="base_link"/>
-    <child link="base_link_spacer_1"/>
-    <origin xyz="${body_x/2} ${body_y/2} 0"
-            rpy="0 0 0"/>
-    <axis xyz="0 0 0"/>
-  </joint>
-  <link name="base_link_spacer_1">
-    <visual>
-      <origin xyz="-${spacer_rud40} -${spacer_rud40} ${spacer_len40/2 + body_z/2}"
-              rpy="0 0 0"/>
-      <geometry>
-        <cylinder length="${spacer_len40}" radius="${spacer_rud40}"/>
-      </geometry>
-      <material name="white">
-        <color rgba="1 1 1 1"/>
-      </material>
-    </visual>
-    <collision>
-      <origin xyz="-${spacer_rud40} -${spacer_rud40} ${spacer_len40/2 + body_z/2}"
-              rpy="0 0 0"/>
-      <geometry>
-        <cylinder length="${spacer_len40}" radius="${spacer_rud40}"/>
-      </geometry>
-    </collision>
-    <inertial>
-      <origin rpy="0 0 0" xyz="0 0 0.5"/>
+  <joint name="base_body_spacer_joint_1" type="fixed">
+    <parent link="base_body"/>
+    <child link="base_body_spacer_1"/>
+    <origin xyz="${body_x/2} ${body_y/2} ${body_z}"
+            rpy="0 0 0"/>
+    <axis xyz="0 0 0"/>
+  </joint>
+  <link name="base_body_spacer_1">
+    <visual>
+      <origin xyz="-${spacer_rud40} -${spacer_rud40} ${spacer_len40/2}"
+              rpy="0 0 0"/>
+      <geometry>
+        <cylinder length="${spacer_len40}" radius="${spacer_rud40}"/>
+      </geometry>
+      <material name="white">
+        <color rgba="1 1 1 1"/>
+      </material>
+    </visual>
+    <collision>
+      <origin xyz="-${spacer_rud40} -${spacer_rud40} ${spacer_len40/2}"
+              rpy="0 0 0"/>
+      <geometry>
+        <cylinder length="${spacer_len40}" radius="${spacer_rud40}"/>
+      </geometry>
+    </collision>
+    <inertial>
+      <origin xyz="-${spacer_rud40} -${spacer_rud40} ${spacer_len40/2}"
+              rpy="0 0 0"/>
       <mass value="0.1"/>
       <inertia ixx="0.1" ixy="0" ixz="0" iyy="0.1" iyz="0" izz="0.1"/>
@@ -114,31 +117,32 @@
   </link>
   <!-- Spacer_2 -->
-  <joint name="base_link_spacer_joint_2" type="fixed">
-    <parent link="base_link"/>
-    <child link="base_link_spacer_2"/>
-    <origin xyz="${body_x/2} -${body_y/2} 0"
-            rpy="0 0 0"/>
-    <axis xyz="0 0 0"/>
-  </joint>
-  <link name="base_link_spacer_2">
-    <visual>
-      <origin xyz="-${spacer_rud40} ${spacer_rud40} ${spacer_len40/2 + body_z/2}"
-              rpy="0 0 0"/>
-      <geometry>
-        <cylinder length="${spacer_len40}" radius="${spacer_rud40}"/>
-      </geometry>
-      <material name="white">
-        <color rgba="1 1 1 1"/>
-      </material>
-    </visual>
-    <collision>
-      <origin xyz="-${spacer_rud40} ${spacer_rud40} ${spacer_len40/2 + body_z/2}"
-              rpy="0 0 0"/>
-      <geometry>
-        <cylinder length="${spacer_len40}" radius="${spacer_rud40}"/>
-      </geometry>
-    </collision>
-    <inertial>
-      <origin rpy="0 0 0" xyz="0 0 0.5"/>
+  <joint name="base_body_spacer_joint_2" type="fixed">
+    <parent link="base_body"/>
+    <child link="base_body_spacer_2"/>
+    <origin xyz="${body_x/2} -${body_y/2} ${body_z}"
+            rpy="0 0 0"/>
+    <axis xyz="0 0 0"/>
+  </joint>
+  <link name="base_body_spacer_2">
+    <visual>
+      <origin xyz="-${spacer_rud40} ${spacer_rud40} ${spacer_len40/2}"
+              rpy="0 0 0"/>
+      <geometry>
+        <cylinder length="${spacer_len40}" radius="${spacer_rud40}"/>
+      </geometry>
+      <material name="white">
+        <color rgba="1 1 1 1"/>
+      </material>
+    </visual>
+    <collision>
+      <origin xyz="-${spacer_rud40} ${spacer_rud40} ${spacer_len40/2}"
+              rpy="0 0 0"/>
+      <geometry>
+        <cylinder length="${spacer_len40}" radius="${spacer_rud40}"/>
+      </geometry>
+    </collision>
+    <inertial>
+      <origin xyz="-${spacer_rud40} ${spacer_rud40} ${spacer_len40/2}"
+              rpy="0 0 0"/>
       <mass value="0.1"/>
       <inertia ixx="0.1" ixy="0" ixz="0" iyy="0.1" iyz="0" izz="0.1"/>
@@ -146,31 +150,32 @@
   </link>
   <!-- Spacer_3 -->
-  <joint name="base_link_spacer_joint_3" type="fixed">
-    <parent link="base_link"/>
-    <child link="base_link_spacer_3"/>
-    <origin xyz="-${body_x/2} ${body_y/2} 0"
-            rpy="0 0 0"/>
-    <axis xyz="0 0 0"/>
-  </joint>
-  <link name="base_link_spacer_3">
-    <visual>
-      <origin xyz="${spacer_rud40} -${spacer_rud40} ${spacer_len40/2 + body_z/2}"
-              rpy="0 0 0"/>
-      <geometry>
-        <cylinder length="${spacer_len40}" radius="${spacer_rud40}"/>
-      </geometry>
-      <material name="white">
-        <color rgba="1 1 1 1"/>
-      </material>
-    </visual>
-    <collision>
-      <origin xyz="${spacer_rud40} -${spacer_rud40} ${spacer_len40/2 + body_z/2}"
-              rpy="0 0 0"/>
-      <geometry>
-        <cylinder length="${spacer_len40}" radius="${spacer_rud40}"/>
-      </geometry>
-    </collision>
-    <inertial>
-      <origin rpy="0 0 0" xyz="0 0 0.5"/>
+  <joint name="base_body_spacer_joint_3" type="fixed">
+    <parent link="base_body"/>
+    <child link="base_body_spacer_3"/>
+    <origin xyz="-${body_x/2} ${body_y/2} ${body_z}"
+            rpy="0 0 0"/>
+    <axis xyz="0 0 0"/>
+  </joint>
+  <link name="base_body_spacer_3">
+    <visual>
+      <origin xyz="${spacer_rud40} -${spacer_rud40} ${spacer_len40/2}"
+              rpy="0 0 0"/>
+      <geometry>
+        <cylinder length="${spacer_len40}" radius="${spacer_rud40}"/>
+      </geometry>
+      <material name="white">
+        <color rgba="1 1 1 1"/>
+      </material>
+    </visual>
+    <collision>
+      <origin xyz="${spacer_rud40} -${spacer_rud40} ${spacer_len40/2}"
+              rpy="0 0 0"/>
+      <geometry>
+        <cylinder length="${spacer_len40}" radius="${spacer_rud40}"/>
+      </geometry>
+    </collision>
+    <inertial>
+      <origin xyz="${spacer_rud40} -${spacer_rud40} ${spacer_len40/2}"
+              rpy="0 0 0"/>
       <mass value="0.1"/>
       <inertia ixx="0.1" ixy="0" ixz="0" iyy="0.1" iyz="0" izz="0.1"/>
@@ -178,31 +183,32 @@
   </link>
   <!-- Spacer_4 -->
-  <joint name="base_link_spacer_joint_4" type="fixed">
-    <parent link="base_link"/>
-    <child link="base_link_spacer_4"/>
-    <origin xyz="-${body_x/2} -${body_y/2} 0"
-            rpy="0 0 0"/>
-    <axis xyz="0 0 0"/>
-  </joint>
-  <link name="base_link_spacer_4">
-    <visual>
-      <origin xyz="${spacer_rud40} ${spacer_rud40} ${spacer_len40/2 + body_z/2}"
-              rpy="0 0 0"/>
-      <geometry>
-        <cylinder length="${spacer_len40}" radius="${spacer_rud40}"/>
-      </geometry>
-      <material name="white">
-        <color rgba="1 1 1 1"/>
-      </material>
-    </visual>
-    <collision>
-      <origin xyz="${spacer_rud40} ${spacer_rud40} ${spacer_len40/2 + body_z/2}"
-              rpy="0 0 0"/>
-      <geometry>
-        <cylinder length="${spacer_len40}" radius="${spacer_rud40}"/>
-      </geometry>
-    </collision>
-    <inertial>
-      <origin rpy="0 0 0" xyz="0 0 0.5"/>
+  <joint name="base_body_spacer_joint_4" type="fixed">
+    <parent link="base_body"/>
+    <child link="base_body_spacer_4"/>
+    <origin xyz="-${body_x/2} -${body_y/2} ${body_z}"
+            rpy="0 0 0"/>
+    <axis xyz="0 0 0"/>
+  </joint>
+  <link name="base_body_spacer_4">
+    <visual>
+      <origin xyz="${spacer_rud40} ${spacer_rud40} ${spacer_len40/2}"
+              rpy="0 0 0"/>
+      <geometry>
+        <cylinder length="${spacer_len40}" radius="${spacer_rud40}"/>
+      </geometry>
+      <material name="white">
+        <color rgba="1 1 1 1"/>
+      </material>
+    </visual>
+    <collision>
+      <origin xyz="${spacer_rud40} ${spacer_rud40} ${spacer_len40/2}"
+              rpy="0 0 0"/>
+      <geometry>
+        <cylinder length="${spacer_len40}" radius="${spacer_rud40}"/>
+      </geometry>
+    </collision>
+    <inertial>
+      <origin xyz="${spacer_rud40} ${spacer_rud40} ${spacer_len40/2}"
+              rpy="0 0 0"/>
       <mass value="0.1"/>
       <inertia ixx="0.1" ixy="0" ixz="0" iyy="0.1" iyz="0" izz="0.1"/>

File: slambot_sim/slambot_description/urdf/slam_robot.urdf (robot description, URDF)
Before this commit: robot slambot, 2 links, 1 joints
Links:
- removed link base_body
Joints:
- removed joint base_footprint_joint

Commit message: update gazebo

File: slambot_sim/slambot_description/urdf/body/body.urdf.xacro (robot description, xacro)
@@ -3,4 +3,5 @@
   <xacro:include filename="$(find slambot_description)/urdf/common_properties.urdf.xacro"/>
   <xacro:include filename="$(find slambot_description)/urdf/body/caster_board.urdf.xacro" />
+  <xacro:include filename="$(find slambot_description)/urdf/body/body.gazebo.xacro" />
   <xacro:property name="tread_width" value="0.1500" />
   <!-- Base Body -->
@@ -15,5 +16,5 @@
   <xacro:macro name="body" params="parent *joint_origin">
   <joint name="base_joint" type="fixed">
-    <insert_block name="joint_origin"/>
+    <xacro:insert_block name="joint_origin"/>
     <parent link="${parent}"/>
     <child link="base_body"/>

File: slambot_sim/slambot_description/urdf/body/caster_board.urdf.xacro (robot description, xacro)
@@ -11,6 +11,6 @@
   <!-- Front caster_board -->
   <joint name="${prefix}_caster_board_joint" type="fixed">
-    <insert_block name="joint_origin"/>
-    <insert_block name="joint_axis"/>
+    <xacro:insert_block name="joint_origin"/>
+    <xacro:insert_block name="joint_axis"/>
     <parent link="${parent}"/>
     <child link="${prefix}_caster_board"/>

File: slambot_sim/slambot_description/urdf/sensors/xtion_pro_live/xtion_pro_live.urdf.xacro (robot description, xacro)
@@ -1,8 +1,6 @@
 <?xml version="1.0"?>
 <robot xmlns:xacro="http://ros.org/wiki/xacro">
-  <!--
-  <xacro:include filename="$(find slabot_description)/urdf/slambot_gazebo.urdf.xacro"/>
-  -->
   <xacro:include filename="$(find slambot_description)/urdf/common_properties.urdf.xacro"/>
+  <xacro:include filename="$(find slambot_description)/urdf/sensors/xtion_pro_live/xtion_pro_live_gazebo.urdf.xacro"/>
   <!-- Xacro properties -->
   <xacro:property name="M_SCALE" value="0.001"/>
@@ -12,6 +10,6 @@
   <xacro:macro name="sensor_xtion_pro_live" params="prefix parent *joint_origin *joint_axis">
     <joint name="${prefix}_rgb_joint" type="fixed">
-      <insert_block name="joint_origin"/>
-      <insert_block name="joint_axis"/>
+      <xacro:insert_block name="joint_origin"/>
+      <xacro:insert_block name="joint_axis"/>
       <parent link="${parent}"/>
       <child link="${prefix}_rgb_frame" />
@@ -86,5 +84,5 @@
         <origin xyz="0 0 0" rpy="${-M_PI/2} 0 0"/>
         <geometry>
-          <mesh filename="package://slabot_description/meshes/sensors/xtion_pro_stack.dae"/>
+          <mesh filename="package://slambot_description/meshes/sensors/xtion_pro_stack.dae"/>
         </geometry>
       </visual>

File: slambot_sim/slambot_description/urdf/slambot.urdf.xacro (robot description, xacro)
@@ -41,5 +41,18 @@
   <!-- <xacro:wheel_trans prefix="right" interface="EffortJointInterface"/> -->
   <!-- <xacro:wheel_trans prefix="left" interface="EffortJointInterface"/> -->
-  <xacro:wheel_trans prefix="right" interface="VelocityJointInterface"/>
-  <xacro:wheel_trans prefix="left" interface="VelocityJointInterface"/>
+  <xacro:wheel_trans prefix="right" interface="VelocityJointInterface" reduction="1.0"/>
+  <xacro:wheel_trans prefix="left" interface="VelocityJointInterface" reduction="1.0"/>
+  <!-- =============== Gazebo =============== -->
+  <gazebo>
+    <plugin name="gazebo_ros_control" filename="libgazebo_ros_control.so">
+      <robotNamespace>slambot</robotNamespace>
+    </plugin>
+  </gazebo>
+  <!-- Body -->
+  <xacro:body_gazebo/>
+  <!-- Wheel -->
+  <xacro:wheel_gazebo prefix="right"/>
+  <xacro:wheel_gazebo prefix="left"/>
+  <!-- Sensors -->
+  <xacro:xtion_pro_live_gazebo camera_name="xtion"/>
 </robot>

File: slambot_sim/slambot_description/urdf/wheel/wheel.transmission.xacro (robot description, xacro)
@@ -1,5 +1,5 @@
 <?xml version="1.0"?>
 <robot xmlns:xacro="http://ros.org/wiki/xacro">
-  <xacro:macro name="wheel_trans" params="prefix interface">
+  <xacro:macro name="wheel_trans" params="prefix interface reduction">
   <transmission name="${prefix}_wheel_trans">
     <type>transmission_interface/SimpleTransmission</type>
@@ -8,4 +8,5 @@
     </joint>
     <actuator name="${prefix}_wheel_motor">
+      <mechanicalReduction>${reduction}</mechanicalReduction>
       <hardwareInterface>${interface}</hardwareInterface>
     </actuator>

File: slambot_sim/slambot_description/urdf/wheel/wheel.urdf.xacro (robot description, xacro)
@@ -7,9 +7,9 @@
   <xacro:property name="wheel_length" value="0.008" />
   <xacro:property name="wheel_mass" value="0.0113"/>
-  <!-- <property name="wheel_radius" value="0.0239"/> -->
+  <!-- <xacro:property name="wheel_radius" value="0.0239"/> -->
   <xacro:macro name="wheel" params="prefix parent *joint_origin *joint_axis">
   <joint name="${prefix}_wheel_joint" type="continuous">
-    <insert_block name="joint_origin"/>
-    <insert_block name="joint_axis"/>
+    <xacro:insert_block name="joint_origin"/>
+    <xacro:insert_block name="joint_axis"/>
     <parent link="${parent}"/>
     <child link="${prefix}_wheel"/>
@@ -25,5 +25,5 @@
     </visual>
     <collision>
-      <!-- <insert_block name="joint_origin"/> -->
+      <!-- <xacro:insert_block name="joint_origin"/> -->
         <geometry>
           <!-- <cylinder radius="${wheel_radius}" length="${wheel_length}"/> -->
