Commit message: update

File: slambot_sim/slambot_description/urdf/body/body.urdf.xacro (robot description, xacro)
@@ -4,4 +4,5 @@
   <xacro:include filename="$(find slambot_description)/urdf/body/caster_board.urdf.xacro" />
   <xacro:include filename="$(find slambot_description)/urdf/body/body.gazebo.xacro" />
+  <xacro:include filename="$(find slambot_description)/urdf/body/spacer.urdf.xacro" />
   <xacro:property name="tread_width" value="0.1500" />
   <!-- Base Body -->
@@ -13,4 +14,5 @@
   <xacro:property name="spacer_len40" value="0.040" />
   <xacro:property name="spacer_rud40" value="0.003" />
+  <xacro:property name="spacer_radius" value="0.003" />
   <xacro:property name="velocity_scale_factor" value="1.0"/>
   <xacro:macro name="body" params="parent *joint_origin">
@@ -85,135 +87,27 @@
   </xacro:caster_board>
   <!-- Spacer_1 -->
-  <joint name="base_body_spacer_joint_1" type="fixed">
-    <parent link="base_body"/>
-    <child link="base_body_spacer_1"/>
-    <origin xyz="${body_x/2} ${body_y/2} ${body_z}"
+  <xacro:spacer prefix="base_body" suffix="1" len="0.040" rad="${spacer_radius}" parent="base_body">
+    <origin xyz="${body_x/2 - spacer_radius} ${body_y/2 - spacer_radius} ${body_z}"
             rpy="0 0 0"/>
     <axis xyz="0 0 0"/>
-  </joint>
-  <link name="base_body_spacer_1">
-    <visual>
-      <origin xyz="-${spacer_rud40} -${spacer_rud40} ${spacer_len40/2}"
-              rpy="0 0 0"/>
-      <geometry>
-        <cylinder length="${spacer_len40}" radius="${spacer_rud40}"/>
-      </geometry>
-      <material name="white">
-        <color rgba="1 1 1 1"/>
-      </material>
-    </visual>
-    <collision>
-      <origin xyz="-${spacer_rud40} -${spacer_rud40} ${spacer_len40/2}"
-              rpy="0 0 0"/>
-      <geometry>
-        <cylinder length="${spacer_len40}" radius="${spacer_rud40}"/>
-      </geometry>
-    </collision>
-    <inertial>
-      <origin xyz="-${spacer_rud40} -${spacer_rud40} ${spacer_len40/2}"
-              rpy="0 0 0"/>
-      <mass value="0.1"/>
-      <inertia ixx="0.1" ixy="0" ixz="0" iyy="0.1" iyz="0" izz="0.1"/>
-    </inertial>
-  </link>
+  </xacro:spacer>
   <!-- Spacer_2 -->
-  <joint name="base_body_spacer_joint_2" type="fixed">
-    <parent link="base_body"/>
-    <child link="base_body_spacer_2"/>
-    <origin xyz="${body_x/2} -${body_y/2} ${body_z}"
+  <xacro:spacer prefix="base_body" suffix="2" len="0.040" rad="${spacer_radius}" parent="base_body">
+    <origin xyz="${body_x/2 - spacer_radius} -${body_y/2 - spacer_radius} ${body_z}"
             rpy="0 0 0"/>
     <axis xyz="0 0 0"/>
-  </joint>
-  <link name="base_body_spacer_2">
-    <visual>
-      <origin xyz="-${spacer_rud40} ${spacer_rud40} ${spacer_len40/2}"
-              rpy="0 0 0"/>
-      <geometry>
-        <cylinder length="${spacer_len40}" radius="${spacer_rud40}"/>
-      </geometry>
-      <material name="white">
-        <color rgba="1 1 1 1"/>
-      </material>
-    </visual>
-    <collision>
-      <origin xyz="-${spacer_rud40} ${spacer_rud40} ${spacer_len40/2}"
-              rpy="0 0 0"/>
-      <geometry>
-        <cylinder length="${spacer_len40}" radius="${spacer_rud40}"/>
-      </geometry>
-    </collision>
-    <inertial>
-      <origin xyz="-${spacer_rud40} ${spacer_rud40} ${spacer_len40/2}"
-              rpy="0 0 0"/>
-      <mass value="0.1"/>
-      <inertia ixx="0.1" ixy="0" ixz="0" iyy="0.1" iyz="0" izz="0.1"/>
-    </inertial>
-  </link>
+  </xacro:spacer>
   <!-- Spacer_3 -->
-  <joint name="base_body_spacer_joint_3" type="fixed">
-    <parent link="base_body"/>
-    <child link="base_body_spacer_3"/>
-    <origin xyz="-${body_x/2} ${body_y/2} ${body_z}"
+  <xacro:spacer prefix="base_body" suffix="3" len="0.040" rad="${spacer_radius}" parent="base_body">
+    <origin xyz="-${body_x/2 - spacer_radius} ${body_y/2 - spacer_radius} ${body_z}"
             rpy="0 0 0"/>
     <axis xyz="0 0 0"/>
-  </joint>
-  <link name="base_body_spacer_3">
-    <visual>
-      <origin xyz="${spacer_rud40} -${spacer_rud40} ${spacer_len40/2}"
-              rpy="0 0 0"/>
-      <geometry>
-        <cylinder length="${spacer_len40}" radius="${spacer_rud40}"/>
-      </geometry>
-      <material name="white">
-        <color rgba="1 1 1 1"/>
-      </material>
-    </visual>
-    <collision>
-      <origin xyz="${spacer_rud40} -${spacer_rud40} ${spacer_len40/2}"
-              rpy="0 0 0"/>
-      <geometry>
-        <cylinder length="${spacer_len40}" radius="${spacer_rud40}"/>
-      </geometry>
-    </collision>
-    <inertial>
-      <origin xyz="${spacer_rud40} -${spacer_rud40} ${spacer_len40/2}"
-              rpy="0 0 0"/>
-      <mass value="0.1"/>
-      <inertia ixx="0.1" ixy="0" ixz="0" iyy="0.1" iyz="0" izz="0.1"/>
-    </inertial>
-  </link>
+  </xacro:spacer>
   <!-- Spacer_4 -->
-  <joint name="base_body_spacer_joint_4" type="fixed">
-    <parent link="base_body"/>
-    <child link="base_body_spacer_4"/>
-    <origin xyz="-${body_x/2} -${body_y/2} ${body_z}"
+  <xacro:spacer prefix="base_body" suffix="4" len="0.040" rad="${spacer_radius}" parent="base_body">
+    <origin xyz="-${body_x/2 - spacer_radius} -${body_y/2 - spacer_radius} ${body_z}"
             rpy="0 0 0"/>
     <axis xyz="0 0 0"/>
-  </joint>
-  <link name="base_body_spacer_4">
-    <visual>
-      <origin xyz="${spacer_rud40} ${spacer_rud40} ${spacer_len40/2}"
-              rpy="0 0 0"/>
-      <geometry>
-        <cylinder length="${spacer_len40}" radius="${spacer_rud40}"/>
-      </geometry>
-      <material name="white">
-        <color rgba="1 1 1 1"/>
-      </material>
-    </visual>
-    <collision>
-      <origin xyz="${spacer_rud40} ${spacer_rud40} ${spacer_len40/2}"
-              rpy="0 0 0"/>
-      <geometry>
-        <cylinder length="${spacer_len40}" radius="${spacer_rud40}"/>
-      </geometry>
-    </collision>
-    <inertial>
-      <origin xyz="${spacer_rud40} ${spacer_rud40} ${spacer_len40/2}"
-              rpy="0 0 0"/>
-      <mass value="0.1"/>
-      <inertia ixx="0.1" ixy="0" ixz="0" iyy="0.1" iyz="0" izz="0.1"/>
-    </inertial>
-  </link>
+  </xacro:spacer>
   </xacro:macro>
 </robot>

Commit message: update

File: slambot_sim/slambot_description/urdf/body/body.urdf.xacro (robot description, xacro)
@@ -10,9 +10,7 @@
   <xacro:property name="body_y" value="0.160" />
   <xacro:property name="body_z" value="0.003" />
-  <xacro:property name="spacer_len27" value="0.027" />
   <xacro:property name="spacer_rud27" value="0.003" />
   <xacro:property name="spacer_len40" value="0.040" />
   <xacro:property name="spacer_rud40" value="0.003" />
-  <xacro:property name="spacer_radius" value="0.003" />
   <xacro:property name="velocity_scale_factor" value="1.0"/>
   <xacro:macro name="body" params="parent *joint_origin">
@@ -87,5 +85,5 @@
   </xacro:caster_board>
   <!-- Spacer_1 -->
-  <xacro:spacer prefix="base_body" suffix="1" len="0.040" rad="${spacer_radius}" parent="base_body">
+  <xacro:spacer prefix="base_body" suffix="1" len="${spacer_len40}" rad="${spacer_radius}" parent="base_body">
     <origin xyz="${body_x/2 - spacer_radius} ${body_y/2 - spacer_radius} ${body_z}"
             rpy="0 0 0"/>
@@ -93,5 +91,5 @@
   </xacro:spacer>
   <!-- Spacer_2 -->
-  <xacro:spacer prefix="base_body" suffix="2" len="0.040" rad="${spacer_radius}" parent="base_body">
+  <xacro:spacer prefix="base_body" suffix="2" len="${spacer_len40}" rad="${spacer_radius}" parent="base_body">
     <origin xyz="${body_x/2 - spacer_radius} -${body_y/2 - spacer_radius} ${body_z}"
             rpy="0 0 0"/>
@@ -99,5 +97,5 @@
   </xacro:spacer>
   <!-- Spacer_3 -->
-  <xacro:spacer prefix="base_body" suffix="3" len="0.040" rad="${spacer_radius}" parent="base_body">
+  <xacro:spacer prefix="base_body" suffix="3" len="${spacer_len40}" rad="${spacer_radius}" parent="base_body">
     <origin xyz="-${body_x/2 - spacer_radius} ${body_y/2 - spacer_radius} ${body_z}"
             rpy="0 0 0"/>
@@ -105,5 +103,5 @@
   </xacro:spacer>
   <!-- Spacer_4 -->
-  <xacro:spacer prefix="base_body" suffix="4" len="0.040" rad="${spacer_radius}" parent="base_body">
+  <xacro:spacer prefix="base_body" suffix="4" len="${spacer_len40}" rad="${spacer_radius}" parent="base_body">
     <origin xyz="-${body_x/2 - spacer_radius} -${body_y/2 - spacer_radius} ${body_z}"
             rpy="0 0 0"/>

File: slambot_sim/slambot_description/urdf/body/caster_board.urdf.xacro (robot description, xacro)
@@ -6,4 +6,5 @@
   <xacro:property name="caster_board_y" value="${body_y}" />
   <xacro:property name="caster_board_z" value="0.003" />
+  <xacro:property name="spacer_len27" value="0.027" />
   <xacro:property name="sphere_radius" value="0.012" />
   <xacro:property name="velocity_scale_factor" value="1.0"/>
@@ -71,131 +72,27 @@
   </link>
   <!-- Spacer_1 -->
-  <joint name="${prefix}_spacer_joint_1" type="fixed">
-    <parent link="${prefix}_caster_board"/>
-    <child link="${prefix}_spacer_1"/>
-    <origin xyz="${caster_board_x/2} ${caster_board_y/2} 0"
+  <xacro:spacer prefix="${prefix}" suffix="1" len="${spacer_len27}" rad="${spacer_radius}" parent="${prefix}_caster_board">
+    <origin xyz="${caster_board_x/2 - spacer_radius} ${caster_board_y/2 - spacer_radius} 0"
             rpy="0 0 0"/>
     <axis xyz="0 0 0"/>
-  </joint>
-  <link name="${prefix}_spacer_1">
-    <visual>
-      <origin xyz="-${spacer_rud27} -${spacer_rud27} ${spacer_len27/2 + caster_board_z/2}"
-              rpy="0 0 0"/>
-      <geometry>
-        <cylinder length="${spacer_len27}" radius="${spacer_rud27}"/>
-      </geometry>
-      <material name="white">
-        <color rgba="1 1 1 1"/>
-      </material>
-    </visual>
-    <collision>
-      <origin xyz="-${spacer_rud27} -${spacer_rud27} ${spacer_len27/2 + caster_board_z/2}"
-              rpy="0 0 0"/>
-      <geometry>
-        <cylinder length="${spacer_len27}" radius="${spacer_rud27}"/>
-      </geometry>
-    </collision>
-    <inertial>
-      <origin rpy="0 0 0" xyz="0 0 0.5"/>
-      <mass value="0.1"/>
-      <inertia ixx="0.1" ixy="0" ixz="0" iyy="0.1" iyz="0" izz="0.1"/>
-    </inertial>
-  </link>
+  </xacro:spacer>
   <!-- Spacer_2 -->
-  <joint name="${prefix}_spacer_joint_2" type="fixed">
-    <parent link="${prefix}_caster_board"/>
-    <child link="${prefix}_spacer_2"/>
-    <origin xyz="${caster_board_x/2} -${caster_board_y/2} 0"
+  <xacro:spacer prefix="${prefix}" suffix="2" len="${spacer_len27}" rad="${spacer_radius}" parent="${prefix}_caster_board">
+    <origin xyz="${caster_board_x/2 - spacer_radius} -${caster_board_y/2 - spacer_radius} 0"
             rpy="0 0 0"/>
     <axis xyz="0 0 0"/>
-  </joint>
-  <link name="${prefix}_spacer_2">
-    <visual>
-      <origin xyz="-${spacer_rud27} ${spacer_rud27} ${spacer_len27/2 + caster_board_z/2}"
-              rpy="0 0 0"/>
-      <geometry>
-        <cylinder length="${spacer_len27}" radius="${spacer_rud27}"/>
-      </geometry>
-      <material name="white">
-        <color rgba="1 1 1 1"/>
-      </material>
-    </visual>
-    <collision>
-      <origin xyz="-${spacer_rud27} ${spacer_rud27} ${spacer_len27/2 + caster_board_z/2}"
-              rpy="0 0 0"/>
-      <geometry>
-        <cylinder length="${spacer_len27}" radius="${spacer_rud27}"/>
-      </geometry>
-    </collision>
-    <inertial>
-      <origin rpy="0 0 0" xyz="0 0 0.5"/>
-      <mass value="0.1"/>
-      <inertia ixx="0.1" ixy="0" ixz="0" iyy="0.1" iyz="0" izz="0.1"/>
-    </inertial>
-  </link>
+  </xacro:spacer>
   <!-- Spacer_3 -->
-  <joint name="${prefix}_spacer_joint_3" type="fixed">
-    <parent link="${prefix}_caster_board"/>
-    <child link="${prefix}_spacer_3"/>
-    <origin xyz="-${caster_board_x/2} ${caster_board_y/2} 0"
+  <xacro:spacer prefix="${prefix}" suffix="3" len="${spacer_len27}" rad="${spacer_radius}" parent="${prefix}_caster_board">
+    <origin xyz="-${caster_board_x/2 - spacer_radius} ${caster_board_y/2 - spacer_radius} 0"
             rpy="0 0 0"/>
     <axis xyz="0 0 0"/>
-  </joint>
-  <link name="${prefix}_spacer_3">
-    <visual>
-      <origin xyz="${spacer_rud27} -${spacer_rud27} ${spacer_len27/2 + caster_board_z/2}"
-              rpy="0 0 0"/>
-      <geometry>
-        <cylinder length="${spacer_len27}" radius="${spacer_rud27}"/>
-      </geometry>
-      <material name="white">
-        <color rgba="1 1 1 1"/>
-      </material>
-    </visual>
-    <collision>
-      <origin xyz="${spacer_rud27} -${spacer_rud27} ${spacer_len27/2 + caster_board_z/2}"
-              rpy="0 0 0"/>
-      <geometry>
-        <cylinder length="${spacer_len27}" radius="${spacer_rud27}"/>
-      </geometry>
-    </collision>
-    <inertial>
-      <origin rpy="0 0 0" xyz="0 0 0.5"/>
-      <mass value="0.1"/>
-      <inertia ixx="0.1" ixy="0" ixz="0" iyy="0.1" iyz="0" izz="0.1"/>
-    </inertial>
-  </link>
+  </xacro:spacer>
   <!-- Spacer_4 -->
-  <joint name="${prefix}_spacer_joint_4" type="fixed">
-    <parent link="${prefix}_caster_board"/>
-    <child link="${prefix}_spacer_4"/>
-    <origin xyz="-${caster_board_x/2} -${caster_board_y/2} 0"
+  <xacro:spacer prefix="${prefix}" suffix="4" len="${spacer_len27}" rad="${spacer_radius}" parent="${prefix}_caster_board">
+    <origin xyz="-${caster_board_x/2 - spacer_radius} -${caster_board_y/2 - spacer_radius} 0"
             rpy="0 0 0"/>
     <axis xyz="0 0 0"/>
-  </joint>
-  <link name="${prefix}_spacer_4">
-    <visual>
-      <origin xyz="${spacer_rud27} ${spacer_rud27} ${spacer_len27/2 + caster_board_z/2}"
-              rpy="0 0 0"/>
-      <geometry>
-        <cylinder length="${spacer_len27}" radius="${spacer_rud27}"/>
-      </geometry>
-      <material name="white">
-        <color rgba="1 1 1 1"/>
-      </material>
-    </visual>
-    <collision>
-      <origin xyz="${spacer_rud27} ${spacer_rud27} ${spacer_len27/2 + caster_board_z/2}"
-              rpy="0 0 0"/>
-      <geometry>
-        <cylinder length="${spacer_len27}" radius="${spacer_rud27}"/>
-      </geometry>
-    </collision>
-    <inertial>
-      <origin rpy="0 0 0" xyz="0 0 0.5"/>
-      <mass value="0.1"/>
-      <inertia ixx="0.1" ixy="0" ixz="0" iyy="0.1" iyz="0" izz="0.1"/>
-    </inertial>
-  </link>
+  </xacro:spacer>
   </xacro:macro>
 </robot>

File: slambot_sim/slambot_description/urdf/common_properties.urdf.xacro (robot description, xacro)
@@ -5,4 +5,5 @@
 <robot name="xacro_properties" xmlns:xacro="http://ros.org/wiki/xacro">
   <xacro:property name="M_PI" value="3.1415926535897931" />
+  <xacro:property name="spacer_radius" value="0.003" />
   <xacro:property name="material_white">
     <material name="white">

Commit message: update

File: slambot_sim/slambot_description/urdf/body/body.urdf.xacro (robot description, xacro)
@@ -10,7 +10,4 @@
   <xacro:property name="body_y" value="0.160" />
   <xacro:property name="body_z" value="0.003" />
-  <xacro:property name="spacer_rud27" value="0.003" />
-  <xacro:property name="spacer_len40" value="0.040" />
-  <xacro:property name="spacer_rud40" value="0.003" />
   <xacro:property name="velocity_scale_factor" value="1.0"/>
   <xacro:macro name="body" params="parent *joint_origin">

File: slambot_sim/slambot_description/urdf/body/caster_board.urdf.xacro (robot description, xacro)
@@ -6,5 +6,4 @@
   <xacro:property name="caster_board_y" value="${body_y}" />
   <xacro:property name="caster_board_z" value="0.003" />
-  <xacro:property name="spacer_len27" value="0.027" />
   <xacro:property name="sphere_radius" value="0.012" />
   <xacro:property name="velocity_scale_factor" value="1.0"/>

File: slambot_sim/slambot_description/urdf/common_properties.urdf.xacro (robot description, xacro)
@@ -6,4 +6,6 @@
   <xacro:property name="M_PI" value="3.1415926535897931" />
   <xacro:property name="spacer_radius" value="0.003" />
+  <xacro:property name="spacer_len27" value="0.027" />
+  <xacro:property name="spacer_len40" value="0.040" />
   <xacro:property name="material_white">
     <material name="white">

Commit message: bug fix

File: slambot_sim/slambot_description/urdf/body/body.urdf.xacro (robot description, xacro)
@@ -71,5 +71,5 @@
   <!-- Front caster_board -->
   <xacro:caster_board prefix="front" parent="base_body">
-    <origin xyz="${body_x/2 - caster_board_x/2} 0 -${spacer_len27}"
+    <origin xyz="${body_x/2 - caster_board_x/2} 0 -${spacer_len27 + body_z/2}"
             rpy="0 0 0"/>
     <axis xyz="0 0 0"/>
@@ -77,5 +77,5 @@
   <!-- Rear caster_board -->
   <xacro:caster_board prefix="rear" parent="base_body">
-    <origin xyz="-${body_x/2 - caster_board_x/2} 0 -${spacer_len27}"
+    <origin xyz="-${body_x/2 - caster_board_x/2} 0 -${spacer_len27 + body_z/2}"
             rpy="0 0 0"/>
     <axis xyz="0 0 0"/>

File: slambot_sim/slambot_description/urdf/body/caster_board.urdf.xacro (robot description, xacro)
@@ -5,9 +5,9 @@
   <xacro:property name="caster_board_x" value="0.060" />
   <xacro:property name="caster_board_y" value="${body_y}" />
-  <xacro:property name="caster_board_z" value="0.003" />
+  <xacro:property name="caster_board_z" value="${body_z}" />
   <xacro:property name="sphere_radius" value="0.012" />
   <xacro:property name="velocity_scale_factor" value="1.0"/>
   <xacro:macro name="caster_board" params="prefix parent *joint_origin *joint_axis">
-  <!-- Front caster_board -->
+  <!-- caster_board -->
   <joint name="${prefix}_caster_board_joint" type="fixed">
     <xacro:insert_block name="joint_origin"/>
@@ -15,7 +15,4 @@
     <parent link="${parent}"/>
     <child link="${prefix}_caster_board"/>
-    <origin xyz="0 0 0"
-            rpy="0 0 0"/>
-    <axis xyz="0 0 0"/>
   </joint>
   <link name="${prefix}_caster_board">
@@ -43,9 +40,9 @@
     <parent link="${prefix}_caster_board"/>
     <child link="${prefix}_caster"/>
-    <origin xyz="0 0 -${sphere_radius}"/>
+    <origin xyz="0 0 -${sphere_radius + caster_board_z/2}"/>
   </joint>
   <link name="${prefix}_caster">
     <visual>
-      <origin xyz="0 0 -${caster_board_z/2}"
+      <origin xyz="0 0 0"
               rpy="0 0 0"/>
       <geometry>
@@ -57,5 +54,5 @@
     </visual>
     <collision>
-      <origin xyz="0 0 -${caster_board_z/2}"
+      <origin xyz="0 0 0"
               rpy="0 0 0"/>
       <geometry>
@@ -64,5 +61,5 @@
     </collision>
     <inertial>
-      <origin xyz="0 0 -${caster_board_z/2}"
+      <origin xyz="0 0 0"
               rpy="0 0 0"/>
       <mass value="0.001"/>
@@ -72,5 +69,5 @@
   <!-- Spacer_1 -->
   <xacro:spacer prefix="${prefix}" suffix="1" len="${spacer_len27}" rad="${spacer_radius}" parent="${prefix}_caster_board">
-    <origin xyz="${caster_board_x/2 - spacer_radius} ${caster_board_y/2 - spacer_radius} 0"
+    <origin xyz="${caster_board_x/2 - spacer_radius} ${caster_board_y/2 - spacer_radius} ${caster_board_z/2}"
             rpy="0 0 0"/>
     <axis xyz="0 0 0"/>
@@ -78,5 +75,5 @@
   <!-- Spacer_2 -->
   <xacro:spacer prefix="${prefix}" suffix="2" len="${spacer_len27}" rad="${spacer_radius}" parent="${prefix}_caster_board">
-    <origin xyz="${caster_board_x/2 - spacer_radius} -${caster_board_y/2 - spacer_radius} 0"
+    <origin xyz="${caster_board_x/2 - spacer_radius} -${caster_board_y/2 - spacer_radius} ${caster_board_z/2}"
             rpy="0 0 0"/>
     <axis xyz="0 0 0"/>
@@ -84,5 +81,5 @@
   <!-- Spacer_3 -->
   <xacro:spacer prefix="${prefix}" suffix="3" len="${spacer_len27}" rad="${spacer_radius}" parent="${prefix}_caster_board">
-    <origin xyz="-${caster_board_x/2 - spacer_radius} ${caster_board_y/2 - spacer_radius} 0"
+    <origin xyz="-${caster_board_x/2 - spacer_radius} ${caster_board_y/2 - spacer_radius} ${caster_board_z/2}"
             rpy="0 0 0"/>
     <axis xyz="0 0 0"/>
@@ -90,5 +87,5 @@
   <!-- Spacer_4 -->
   <xacro:spacer prefix="${prefix}" suffix="4" len="${spacer_len27}" rad="${spacer_radius}" parent="${prefix}_caster_board">
-    <origin xyz="-${caster_board_x/2 - spacer_radius} -${caster_board_y/2 - spacer_radius} 0"
+    <origin xyz="-${caster_board_x/2 - spacer_radius} -${caster_board_y/2 - spacer_radius} ${caster_board_z/2}"
             rpy="0 0 0"/>
     <axis xyz="0 0 0"/>
