Commit message: update

File: slambot_sim/slambot_description/urdf/body/caster_board.urdf.xacro (robot description, xacro)
@@ -56,4 +56,17 @@
       </material>
     </visual>
+    <collision>
+      <origin xyz="0 0 -${caster_board_z/2}"
+              rpy="0 0 0"/>
+      <geometry>
+        <sphere radius="${sphere_radius}"/>
+      </geometry>
+    </collision>
+    <inertial>
+      <origin xyz="0 0 -${caster_board_z/2}"
+              rpy="0 0 0"/>
+      <mass value="0.001"/>
+      <inertia ixx="0.0020833333" ixy="0" ixz="0" iyy="0.0070833333" iyz="0" izz="0.0083333333"/>
+    </inertial>
   </link>
   <!-- Spacer_1 -->

Commit message: bug fix

File: slambot_sim/slambot_description/urdf/body/caster_board.urdf.xacro (robot description, xacro)
@@ -6,5 +6,5 @@
   <xacro:property name="caster_board_y" value="${body_y}" />
   <xacro:property name="caster_board_z" value="${body_z}" />
-  <xacro:property name="sphere_radius" value="0.012" />
+  <xacro:property name="sphere_radius" value="0.01198" />
   <xacro:property name="velocity_scale_factor" value="1.0"/>
   <xacro:macro name="caster_board" params="prefix parent *joint_origin *joint_axis">
