Commit message: update

File: slambot_sim/slambot_description/urdf/slambot.urdf.xacro (robot description, xacro)
@@ -47,5 +47,5 @@
     <plugin name="gazebo_ros_control" filename="libgazebo_ros_control.so">
       <robotNamespace>slambot_host</robotNamespace>
-	  <robotParam>slambot_description</robotParam>
+	  <robotParam>robot_description</robotParam>
     </plugin>
   </gazebo>

File: slambot_sim/slambot_description/urdf/wheel/wheel.urdf.xacro (robot description, xacro)
@@ -27,6 +27,6 @@
       <!-- <xacro:insert_block name="joint_origin"/> -->
         <geometry>
-          <!-- <cylinder radius="${wheel_radius}" length="${wheel_length}"/> -->
-          <mesh filename="package://slambot_description/urdf/wheel/meshes/RasPiMouse_wheel.dae"/>
+          <cylinder radius="${wheel_radius}" length="${wheel_length}"/>
+          <!-- <mesh filename="package://slambot_description/urdf/wheel/meshes/RasPiMouse_wheel.dae"/> -->
         </geometry>
     </collision>
