Commit message: remove limit

File: slambot_description/urdf/wheel/wheel.gazebo.xacro (robot description, xacro)
@@ -11,5 +11,5 @@
       <kd>100.0</kd>
       <minDepth>0.001</minDepth>
-      <maxVel>1.0</maxVel>
+      <!--   <maxVel>1.0</maxVel> -->
     </gazebo>
   </xacro:macro>

File: slambot_description/urdf/wheel/wheel.urdf.xacro (robot description, xacro)
@@ -14,5 +14,5 @@
     <parent link="${parent}"/>
     <child link="${prefix}_wheel"/>
-    <limit effort="70" velocity="15"/>
+    <!-- <limit effort="70" velocity="15"/> -->
     <safety_controller  k_velocity="10" />
     <dynamics damping="1.0" friction="1.0" />
