Commit message: update

File: slambot_description/urdf/sensors/xtion_pro_live/xtion_pro_live.urdf.xacro (robot description, xacro)
@@ -5,5 +5,5 @@
   <!-- Xacro properties -->
   <xacro:property name="M_SCALE" value="0.001"/>
-  <xacro:property name="xtion_pro_live_ir_rel_rgb_py" value="0.0270" />
+  <xacro:property name="xtion_pro_live_dep_rel_rgb_py" value="0.0270" />
   <xacro:property name="xtion_pro_live_cam_rel_rgb_py"   value="-0.0220" />
   <!-- Parameterised in part by the values in slambot_properties.urdf.xacro -->
@@ -55,20 +55,20 @@
     </joint>
     <link name="${prefix}_rgb_optical_frame"/>
-    <!-- Xtion IR sensor physical attachment -->
-    <joint name="${prefix}_ir_joint" type="fixed">
-      <origin xyz="0 ${xtion_pro_live_ir_rel_rgb_py} 0"
+    <!-- Xtion Depth sensor physical attachment -->
+    <joint name="${prefix}_depth_joint" type="fixed">
+      <origin xyz="0 ${xtion_pro_live_dep_rel_rgb_py} 0"
               rpy="0 0 0" />
       <parent link="${prefix}_rgb_frame" />
-      <child link="${prefix}_ir_frame" />
+      <child link="${prefix}_depth_frame" />
     </joint>
-    <link name="${prefix}_ir_frame"/>
-    <!-- Xtion IR sensor frame -->
-    <joint name="${prefix}_ir_optical_joint" type="fixed">
+    <link name="${prefix}_depth_frame"/>
+    <!-- Xtion Depth sensor frame -->
+    <joint name="${prefix}_depth_optical_joint" type="fixed">
       <origin xyz="0 0 0"
               rpy="${-M_PI/2} 0 ${-M_PI/2}" />
-      <parent link="${prefix}_ir_frame" />
-      <child link="${prefix}_ir_optical_frame" />
+      <parent link="${prefix}_depth_frame" />
+      <child link="${prefix}_depth_optical_frame" />
     </joint>
-    <link name="${prefix}_ir_optical_frame"/>
+    <link name="${prefix}_depth_optical_frame"/>
     <!-- RGBD sensor for simulation, same as Kinect -->
     <slambot_sim_3dsensor/>

File: slambot_description/urdf/sensors/xtion_pro_live/xtion_pro_live_gazebo.urdf.xacro (robot description, xacro)
@@ -3,5 +3,5 @@
   <!-- Microsoft Kinect / ASUS Xtion PRO Live for simulation -->
   <xacro:macro name="xtion_pro_live_gazebo" params="camera_name">
-    <gazebo reference="${camera_name}_ir_frame">
+    <gazebo reference="${camera_name}_depth_frame">
       <sensor type="depth" name="${camera_name}">
         <always_on>true</always_on>
@@ -28,5 +28,5 @@
           <cameraInfoTopicName>rgb/camera_info</cameraInfoTopicName>
           <depthImageCameraInfoTopicName>depth_registered/camera_info</depthImageCameraInfoTopicName>
-          <frameName>/${camera_name}_ir_optical_frame</frameName>
+          <frameName>/${camera_name}_depth_optical_frame</frameName>
           <baseline>0.1</baseline>
           <distortion_k1>0.0</distortion_k1>
