Commit message: update

File: slambot_description/urdf/sensors/xtion_pro_live/xtion_pro_live_gazebo.urdf.xacro (robot description, xacro)
@@ -2,5 +2,5 @@
 <robot xmlns:xacro="http://ros.org/wiki/xacro">
   <!-- Microsoft Kinect / ASUS Xtion PRO Live for simulation -->
-  <xacro:macro name="xtion_pro_live_gazebo" params="camera_name">
+  <xacro:macro name="xtion_pro_live_gazebo" params="camera_name name_space">
     <gazebo reference="${camera_name}_depth_frame">
       <sensor type="depth" name="${camera_name}">
@@ -20,4 +20,5 @@
         </camera>
         <plugin name="kinect_${camera_name}_controller" filename="libgazebo_ros_openni_kinect.so">
+          <robotNamespace>${name_space}</robotNamespace>
           <cameraName>${camera_name}</cameraName>
           <alwaysOn>true</alwaysOn>

File: slambot_description/urdf/slambot.urdf.xacro (robot description, xacro)
@@ -55,4 +55,4 @@
   <xacro:wheel_gazebo prefix="left"/>
   <!-- Sensors -->
-  <xacro:xtion_pro_live_gazebo camera_name="xtion_pro_live"/>
+  <xacro:xtion_pro_live_gazebo camera_name="xtion_pro_live" name_space="slambot_sensor"/>
 </robot>
